File: SemuBot_WheelBase/Wheelbase/Wheelbase.kicad_pcb (KiCad board)
At the start: 2 copper layers, 110 x 90 mm, 129 parts, among them IC1 DRV8353FSRTAR, IC2 DRV8353FSRTAR, IC3 DRV8353FSRTAR, IC4 ADS131M03IRUKT, IC5 ADS131M03IRUKT, IC6 ADS131M03IRUKT, J1 10155435-00011LF, J10 B5B-XH-A_LF__SN_, J11 B5B-XH-A_LF__SN_, J12 B5B-XH-A_LF__SN_, J13 MTSW-104-09-L-S-400, J14 XT30PW-M, J15 MTSW-104-09-L-S-400, J2 MTSW-102-09-L-S-400, J3 MR30PW-M, J4 B5B-XH-A_LF__SN_, J5 B5B-XH-A_LF__SN_, J6 B5B-XH-A_LF__SN_, J7 MR30PW-M, J8 MR30PW-M, J9 DS1013-10SSIB1, Q1 AON7262E, Q10 AON7262E, Q11 AON7262E, Q12 AON7262E, Q13 AON7262E, Q14 AON7262E, Q15 AON7262E, Q19 AON7262E, Q2 AON7262E, Q20 AON7262E, Q21 AON7262E, Q3 AON7262E, Q4 AON7262E, Q5 AON7262E, Q6 AON7262E, Q7 AON7262E, Q8 AON7262E, Q9 AON7262E, U1 STM32F303RET6, U5 RT9013-33GB, Y1 ECS-2520MVLC-081.92-CN-TR, Y2 X322516MLB4SI

Commit message: Encoder fix
Parts:
- added C2: 100nF, Capacitor_SMD:C_0603_1608Metric_Pad1.08x0.95mm_HandSolder, F.Cu at (136.5, 65.4)
- added D1: green, LED_SMD:LED_0603_1608Metric_Pad1.05x0.95mm_HandSolder, F.Cu at (145.5, 68.5)
- added R23: 10k, Resistor_SMD:R_0603_1608Metric_Pad0.98x0.95mm_HandSolder, F.Cu at (136.5, 66.8)
- added R24: 100, Resistor_SMD:R_0603_1608Metric_Pad0.98x0.95mm_HandSolder, F.Cu at (136.5, 68.3)
- added R25: 3.3K, Resistor_SMD:R_0603_1608Metric_Pad0.98x0.95mm_HandSolder, F.Cu at (142.1, 68.5)
- added R26: 3.3K, Resistor_SMD:R_0603_1608Metric_Pad0.98x0.95mm_HandSolder, F.Cu at (150.0, 94.5)
- added S1: SWT0211-050010GSA_REVA, switch:SW_SWT0211-050010GSA_REVA, F.Cu at (130.5, 65.8)
- moved R3 3.22 mm to (183.2, 79.8), turned to 90 degrees
- moved C34 2.71 mm to (165.8, 109.1)
- moved D2 2.21 mm to (145.7, 67.0)
- moved R6 2.10 mm to (142.4, 67.0)
- moved C30 1.21 mm to (148.4, 107.8), turned to 0 degrees
- moved R45 0.69 mm to (148.3, 91.8)
- moved C26 0.32 mm to (148.1, 110.3)
- moved C22 0.31 mm to (142.8, 106.6)
- moved J4 0.25 mm to (169.0, 93.5), turned to 90 degrees
Connections:
- IC4 pad 12: /SPI_CLK -> /SPI1_SCK
- IC4 pad 13: /SPI_MOSI -> /SPI1_MISO
- IC4 pad 14: /SPI_DATA -> /SPI1_MOSI
- IC4 pad 19: GND -> +3.3V
- IC5 pad 12: /SPI_CLK -> /SPI1_SCK
- IC5 pad 13: /SPI_MOSI -> /SPI1_MISO
- IC5 pad 14: /SPI_DATA -> /SPI1_MOSI
- IC5 pad 19: GND -> +3.3V
- IC6 pad 12: /SPI_CLK -> /SPI1_SCK
- IC6 pad 13: /SPI_MOSI -> /SPI1_MISO
- IC6 pad 14: /SPI_DATA -> /SPI1_MOSI
- IC6 pad 19: GND -> +3.3V
- J10 pad 2: /SSI_DATA -> /enc_1_data
- J11 pad 2: /SSI_DATA -> /enc_2_data
- J12 pad 2: /SSI_DATA -> /enc_3_data
- J4 pad 2: /Motor_1/HAL_3 -> /Motor_1/HAL_1
- J4 pad 4: /Motor_1/HAL_1 -> /Motor_1/HAL_3
- U1 pad 11: unconnected-(U1-PC3-Pad11) -> /MOTOR1_DIR
- U1 pad 21: /MOTOR2_DIR -> /SPI1_SCK
- U1 pad 22: /MOTOR2_PWM -> /SPI1_MISO
- U1 pad 23: /motor3_nBRAKE -> /SPI1_MOSI
- U1 pad 25: unconnected-(U1-PC5-Pad25) -> /MOTOR2_DIR
- U1 pad 26: unconnected-(U1-PB0-Pad26) -> /motor3_nBRAKE
- U1 pad 3: unconnected-(U1-PC14-Pad3) -> Net-(D1-A)
- U1 pad 37: /MOTOR1_DIR -> /MOTOR2_PWM
- U1 pad 4: unconnected-(U1-PC15-Pad4) -> /enc_2_data
- U1 pad 55: /SSI_DATA -> /enc_1_data
- U1 pad 57: unconnected-(U1-PB5-Pad57) -> /enc_3_data
Routing:
- net /SSI_DATA: track 240.5 -> 0.00 mm, vias 3 -> 0
- net /enc_3_data: track 0.00 -> 146.8 mm, vias 0 -> 4
- net /SPI1_SCK: track 0.00 -> 113.6 mm, vias 0 -> 7
- net /SPI1_MOSI: track 0.00 -> 110.1 mm, vias 0 -> 15
- net /SPI1_MISO: track 0.00 -> 105.2 mm, vias 0 -> 8
- net /enc_2_data: track 0.00 -> 94.1 mm, vias 0 -> 1
- net /enc_1_data: track 0.00 -> 86.9 mm, vias 0 -> 3
- net /SPI_CLK: track 125.2 -> 85.4 mm, vias 12 -> 8
- net /SPI_MOSI: track 128.7 -> 92.5 mm, vias 10 -> 8
- net /NRST: track 33.2 -> 53.3 mm, vias 2 -> 3
- net +3.3V: track 281.9 -> 299.8 mm
- net /SPI_DATA: track 127.6 -> 112.5 mm, vias 13 -> 9
- net /MOTOR1_DIR: track 28.6 -> 40.3 mm
- net Net-(R24-Pad2): track 0.00 -> 8.90 mm
- net /MOTOR2_DIR: track 22.2 -> 31.0 mm, vias 2 -> 4
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Other:
- board text added: "DEBUG2"
- board text added: "RESET"
