File: SemuBot_WheelBase/Wheelbase/Wheelbase.kicad_pcb (KiCad board)
At the start: 4 copper layers, 110 x 90 mm, 130 parts, among them IC1 DRV8353FSRTAR, IC2 DRV8353FSRTAR, IC3 DRV8353FSRTAR, J1 10155435-00011LF, J10 B5B-XH-A_LF__SN_, J11 B5B-XH-A_LF__SN_, J12 B5B-XH-A_LF__SN_, J13 MTSW-104-09-L-S-400, J14 XT30PW-M, J3 MR30PW-M, J4 B5B-XH-A_LF__SN_, J5 B5B-XH-A_LF__SN_, J6 B5B-XH-A_LF__SN_, J7 MR30PW-M, J8 MR30PW-M, J9 DS1013-10SSIB1, Q1 AONR62818, Q10 AONR62818, Q11 AONR62818, Q12 AONR62818, Q13 AONR62818, Q14 AONR62818, Q15 AONR62818, Q19 AONR62818, Q2 AONR62818, Q20 AONR62818, Q21 AONR62818, Q3 AONR62818, Q4 AONR62818, Q5 AONR62818, Q6 AONR62818, Q7 AONR62818, Q8 AONR62818, Q9 AONR62818, U1 STM32G474RET6, U5 RT9013-33GB, Y2 X322516MLB4SI

Commit message: Schematic and pcb fix
Parts:
- moved C50 5.48 mm to (125.3, 118.2), turned to 0 degrees
- moved C51 5.40 mm to (120.2, 121.2), turned to 180 degrees
- moved C52 4.57 mm to (126.7, 131.2), turned to 180 degrees
Connections:
- C50 pad 1: GND -> +24V
- C50 pad 2: +24V -> GND
- C51 pad 1: GND -> +24V
- C51 pad 2: +24V -> GND
- C52 pad 1: GND -> +24V
- C52 pad 2: +24V -> GND
