File: SemuBot_WheelBase/Wheelbase/Driver.kicad_sch (KiCad schematic)
At the start: 27 parts, among them IC1 DRV8353FSRTAR, IC4 ADS131M03IRUKT, Q1 AON7262E, Q19 AON7262E, Q2 AON7262E, Q3 AON7262E, Q5 AON7262E, Q6 AON7262E

Commit message: Re organizing, adding .pdf
Other:
- note added: "ADC for current measuring. DRV8353 outputs measured voltage from the shunt, between SPX/SNX"
- note added: "HALL PullUps"
- moved on the sheet: R29, R32, R35
