File: SemuBot_WheelBase/Wheelbase/Driver.kicad_sch (KiCad schematic)
At the start: 27 parts, among them IC1 DRV8353FSRTAR, IC4 ADS131M03IRUKT, Q1 AON7262E, Q19 AON7262E, Q2 AON7262E, Q3 AON7262E, Q5 AON7262E, Q6 AON7262E

Commit message: New 4-layer board
Parts:
- removed C16: 220nF, Capacitor_SMD:C_0603_1608Metric_Pad1.08x0.95mm_HandSolder, symbol Device:C
- removed C51: 100nF, Capacitor_SMD:C_0603_1608Metric_Pad1.08x0.95mm_HandSolder, symbol Device:C
- removed IC4: ADS131M03IRUKT, QFN40P300X300X80-21N-D, symbol ADS131M03IRUKT:ADS131M03IRUKT
- removed R3: 1.5K, Resistor_SMD:R_0603_1608Metric_Pad0.98x0.95mm_HandSolder, symbol Device:R
- added C41: 1uF 63V, Capacitor_SMD:C_0603_1608Metric_Pad1.08x0.95mm_HandSolder, symbol Device:C
- C35, C38: value 100nF -> 1uF 63V
- Q1, Q19, Q2, Q3, Q5, Q6: value AON7262E -> AONR62818
Connections:
- net +24V: now also Q1.10 (D), Q1.5 (D), Q1.6 (D), Q1.7 (D), Q1.8 (D), Q1.9 (D), Q3.10 (D), Q3.5 (D), Q3.6 (D), Q3.7 (D), Q3.8 (D), Q3.9 (D), Q5.10 (D), Q5.5 (D), Q5.6 (D), Q5.7 (D), Q5.8 (D), Q5.9 (D)
- net +3.3V: no longer C35.1, C38.1
- net GND: now also C41.2; no longer IC1.10 (SNA), IC1.11 (SNB), IC1.20 (SNC), R12.1, R15.1, R9.1
- net MA: now also Q1.1 (S), Q1.2 (S), Q2.10 (D), Q2.5 (D), Q2.6 (D), Q2.7 (D), Q2.8 (D), Q2.9 (D)
- net MB: now also Q19.10 (D), Q19.5 (D), Q19.6 (D), Q19.7 (D), Q19.8 (D), Q19.9 (D), Q3.1 (S), Q3.2 (S)
- net MC: now also Q5.1 (S), Q5.2 (S), Q6.10 (D), Q6.5 (D), Q6.6 (D), Q6.7 (D), Q6.8 (D), Q6.9 (D)
- net SPA: now also Q2.1 (S), Q2.2 (S)
- net SPB: now also Q19.1 (S), Q19.2 (S)
- net SPC: now also Q6.1 (S), Q6.2 (S)
- new net SNA: C35.1, IC1.10 (SNA), R9.1
- new net SNB: C41.1, IC1.11 (SNB), R15.1
- new net SNC: C38.1, IC1.20 (SNC), R12.1
- no-connect marks 2 -> 0
Other:
- note removed: "ADC for current measuring. DRV8353 outputs measured voltage from the shunt, between SPX/SNX"

Commit message: Fixes
Parts:
- removed R4: 3.3K, Resistor_SMD:R_0603_1608Metric_Pad0.98x0.95mm_HandSolder, symbol Device:R
- C35, C38, C41: value 1uF 63V -> 1uF 50V X7R; footprint Capacitor_SMD:C_0603_1608Metric_Pad1.08x0.95mm_HandSolder -> Capacitor_SMD:C_0805_2012Metric_Pad1.18x1.45mm_HandSolder
Connections:
- net +24V: now also C35.1, C38.1, C41.1
- net GND: now also IC1.10 (SNA), IC1.11 (SNB), IC1.20 (SNC), R12.1, R15.1, R9.1
- removed net SNA: C35.1, IC1.10 (SNA), R9.1
- removed net SNB: C41.1, IC1.11 (SNB), R15.1
- removed net SNC: C38.1, IC1.20 (SNC), R12.1
- no-connect marks 0 -> 1
Other:
- moved on the sheet: R9
