File: SemuBot_WheelBase/Wheelbase/Wheelbase.kicad_sch (KiCad schematic)
At the start: 54 parts, among them J1 10155435-00011LF, J10 B5B-XH-A_LF__SN_, J11 B5B-XH-A_LF__SN_, J12 B5B-XH-A_LF__SN_, J13 MTSW-104-09-L-S-400, J14 XT30PW-M, J15 MTSW-104-09-L-S-400, J2 MTSW-102-09-L-S-400, J3 MR30PW-M, J4 B5B-XH-A_LF__SN_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

Commit message: Re organizing, adding .pdf
Other:
- note added: "M3 holes"
- note added: "MCU"
- note added: "SPI PullUps"
- moved on the sheet: D3, H1, H2, H3, H4, J10, J11, J12, J13, J14, J15, J2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
