File: SemuBot_WheelBase/Wheelbase/Wheelbase.kicad_sch (KiCad schematic)
At the start: 54 parts, among them J1 10155435-00011LF, J10 B5B-XH-A_LF__SN_, J11 B5B-XH-A_LF__SN_, J12 B5B-XH-A_LF__SN_, J13 MTSW-104-09-L-S-400, J14 XT30PW-M, J15 MTSW-104-09-L-S-400, J2 MTSW-102-09-L-S-400, J3 MR30PW-M, J4 B5B-XH-A_LF__SN_, J5 B5B-XH-A_LF__SN_, J6 B5B-XH-A_LF__SN_, J7 MR30PW-M, J8 MR30PW-M, J9 DS1013-10SSIB1, U1 STM32F303RET6, U5 RT9013-33GB, Y1 ECS-2520MVLC-081.92-CN-TR, Y2 X322516MLB4SI

Commit message: New 4-layer board
Parts:
- removed C2, C50: 100nF, Capacitor_SMD:C_0603_1608Metric_Pad1.08x0.95mm_HandSolder, symbol Device:C
- removed J15: MTSW-104-09-L-S-400, MTSW-104-09-L-S-400:SAMTEC_MTSW-104-09-L-S-400, symbol MTSW-104-09-L-S-400:MTSW-104-09-L-S-400
- removed J2: MTSW-102-09-L-S-400, MTSW-102-09-L-S-400.:SAMTEC_MTSW-102-09-L-S-400, symbol MTSW-102-09-L-S-400:MTSW-102-09-L-S-400
- removed R23: 10k, Resistor_SMD:R_0603_1608Metric_Pad0.98x0.95mm_HandSolder, symbol Device:R
- removed R24: 100, Resistor_SMD:R_0603_1608Metric_Pad0.98x0.95mm_HandSolder, symbol Device:R
- removed R36: 1.5k, Resistor_SMD:R_0603_1608Metric_Pad0.98x0.95mm_HandSolder, symbol Device:R
- removed S1: SWT0211-050010GSA_REVA, switch:SW_SWT0211-050010GSA_REVA, symbol SWT0211-050010GSA_REVA:SWT0211-050010GSA_REVA
- removed U1: STM32F303RET6, Package_QFP:LQFP-64_10x10mm_P0.5mm, symbol MCU_ST_STM32F3:STM32F303RETx
- removed Y1: ECS-2520MVLC-081.92-CN-TR, ECS-2520:OSC_ECS-2520MVLC-081.92-CN-TR, symbol ECS-2520MVLC-081.92-CN-TR:ECS-2520MVLC-081.92-CN-TR
- added C16, C34, C44, C45, C46: 100nF, Capacitor_SMD:C_0603_1608Metric_Pad1.08x0.95mm_HandSolder, symbol Device:C
- added D4: BZX84C3V3, BZX84C3V3:SOT95P240X115-3N, symbol BZX84C3V3:BZX84C3V3
- added D5: SMCJ33A, SMCJ33A:DIOM6859X262N, symbol SMCJ33A:SMCJ33A
- added R27: 10k, Resistor_SMD:R_0603_1608Metric_Pad0.98x0.95mm_HandSolder, symbol Device:R
- added U1: STM32G474RET6, Package_QFP:LQFP-64_10x10mm_P0.5mm, symbol MCU_ST_STM32G4:STM32G474RETx
- R26: value 3.3K -> 91k
Connections:
- net SPI1_MISO is gone; now on net +24V: R26.1
- net +24V: now also D5.C
- net +3.3V: now also C16.1, C44.1, C45.1, C46.1, U1.1 (VBAT), U1.16 (VDD), U1.28 (VREF+), U1.29 (VDDA), U1.32 (VDD), U1.48 (VDD), U1.64 (VDD); no longer R26.2
- net CAN_RX: now also U1.61 (PB8)
- net CAN_TX: now also U1.62 (PB9)
- net CS_ENC_1: now also U1.56 (PB3)
- net CS_ENC_2: now also U1.9 (PC1)
- net CS_ENC_3: now also U1.41 (PC9)
- net D+: now also U1.46 (PA12)
- net D-: now also U1.45 (PA11)
- net ENABLE: now also U1.30 (PB10)
- net GND: now also C16.2, C34.2, C44.2, C45.2, C46.2, D4.1, D5.A, R27.2, U1.15 (VSS), U1.31 (VSS), U1.47 (VSS), U1.63 (VSS)
- net MOTOR1_DIR: now also U1.43 (PA9)
- net MOTOR1_PWM: now also U1.8 (PC0)
- net MOTOR2_DIR: now also U1.34 (PB12)
- net MOTOR2_PWM: now also U1.51 (PA15)
- net MOTOR3_DIR: now also U1.38 (PC6)
- net MOTOR3_PWM: now also U1.26 (PB2)
- net NRST: now also U1.7 (PG10)
- net OSC_IN: now also U1.5 (PF0)
- net OSC_OUT: now also U1.6 (PF1)
- net SPI3_NSS: now also U1.18 (PA4)
- net SPI_CLK: now also U1.19 (PA5)
- net SPI_DATA: now also U1.57 (PB4)
- net SPI_MOSI: now also U1.58 (PB5)
- net SSI_CLK: now also U1.60 (PB7)
- net SWCLK: now also U1.50 (PA14)
- net SWDIO: now also U1.49 (PA13)
- net enc_1_data: now also U1.59 (PB6)
- net enc_2_data: now also U1.4 (PC15)
- net enc_3_data: now also U1.55 (PD2)
- net motor1_Cs: now also U1.52 (PC10)
- net motor1_nBRAKE: now also U1.42 (PA8)
- net motor2_Cs: now also U1.17 (PA3)
- net motor2_nBRAKE: now also U1.33 (PB11)
- net motor3_Cs: now also U1.37 (PB15)
- net motor3_nBRAKE: now also U1.39 (PC7)
- net at D2.2 (A): now also U1.10 (PC2)
- net at D1.2 (A): now also U1.11 (PC3)
- new net: C34.1, U1.27 (VSSA)
- new net ADC1_IN1: U1.12 (PA0)
- new net ADC1_IN2: U1.13 (PA1)
- new net ADC1_IN3: U1.14 (PA2)
- new net ADC2_IN3: U1.20 (PA6)
- new net ADC2_IN4: U1.21 (PA7)
- new net ADC2_IN5: U1.22 (PC4)
- new net ADC3_IN1: U1.25 (PB1)
- new net ADC3_IN12: U1.24 (PB0)
- new net ADC3_IN5: U1.35 (PB13)
- new net ADC4_IN3: D4.3, R26.2, R27.1, U1.36 (PB14)
- no-connect marks 10 -> 7
Other:
- sheet Motor_1 ports: added SOA, SOB, SOC; removed ADC_CS, DRDY, SPI1_MISO, SPI1_MOSI, SPI1_SCLK, adc_CLK
- sheet Motor_2 ports: added SOA, SOB, SOC; removed ADC_CS, DRDY, SPI1_MISO, SPI1_MOSI, SPI1_SCLK, adc_CLK
- sheet Motor_3 ports: added SOA, SOB, SOC; removed ADC_CS, DRDY, SPI1_MISO, SPI1_MOSI, SPI1_SCLK, adc_CLK
- note removed: "5V input"
- note removed: "CLK signal for ADC"
- note removed: "MCU"
- note removed: "RESET Switch"
- note removed: "SPI"
- moved on the sheet: C12, C13, C14, C15, C3, D2, H1, H2, H3, H4, R6

Commit message: Fixes
Parts:
- added C47, C48, C49, C53: 100nF, Capacitor_SMD:C_0603_1608Metric_Pad1.08x0.95mm_HandSolder, symbol Device:C
- added C50, C51, C52: 470uF 5mm 63V Polymer, Capacitor_THT:CP_Radial_D10.0mm_P5.00mm, symbol Device:C
Connections:
- net +24V: now also C50.2, C51.2, C52.2, C53.1
- net +5V: now also C47.1, C48.1, C49.1
- net GND: now also C47.2, C48.2, C49.2, C50.1, C51.1, C52.1, C53.2
Other:
- moved on the sheet: J14
